Commit message: corrected xacro file and saved Rviz config

File: catkin_ws/src/two_wheel_robo/urdf/two_wheel_robo.xacro (robot description, xacro)
@@ -67,4 +67,5 @@
     </visual>
     <collision>
+      <origin xyz="0 0 0" rpy=" 0 1.5707 1.5707"/>
       <geometry>
         <cylinder length="0.05" radius="0.1"/>
@@ -92,4 +93,5 @@
     </visual>
     <collision>
+      <origin xyz="0 0 0" rpy=" 0 1.5707 1.5707"/>
       <geometry>
         <cylinder length="0.05" radius="0.1"/>
